File: MSX Mega Adapter.kicad_pcb (KiCad board)
At the start: 2 copper layers, 30.5 x 31.8 mm, 8 parts, among them J1 Atari 7800, J2 Mega Drive, Q1 2N3906, Q2 2N3906

Commit message: Layout done
Parts:
- removed Q1, Q2: 2N3906, TO_SOT_Packages_THT:TO-92_Inline_Wide
- removed R1, R3: 620, Resistors_THT:R_Axial_DIN0207_L6.3mm_D2.5mm_P10.16mm_Horizontal
- removed R2, R4: 1k, Resistors_THT:R_Axial_DIN0207_L6.3mm_D2.5mm_P10.16mm_Horizontal
- added C1: 100nF, Capacitors_THT:C_Disc_D4.7mm_W2.5mm_P5.00mm, F.Cu at (134.0, 67.9)
- added D1: 1n5711, Diodes_THT:D_DO-35_SOD27_P7.62mm_Horizontal, F.Cu at (135.3, 61.1)
- added D2: 1n5711, Diodes_THT:D_DO-35_SOD27_P7.62mm_Horizontal, F.Cu at (135.3, 64.8)
- added U1: 74HCT04, Housings_DIP:DIP-14_W7.62mm_Socket_LongPads, F.Cu at (127.6, 71.8)
- J1: value Atari 7800 -> MSX
Connections:
- J1 pad 5: PADDLE_B -> VCC
- J1 pad 6: FIRE -> TRIGGER1
- J1 pad 7: VCC -> TRIGGER2
- J1 pad 8: GND -> OUT
- J1 pad 9: PADDLE_A -> GND
- J2 pad 6: /MD_BTN_B -> Net-(D1-Pad1)
- J2 pad 7: VCC -> Net-(J2-Pad7)
- J2 pad 9: /MD_BTN_C -> Net-(D2-Pad1)
Routing:
- net /MD_BTN_C: track 35.5 -> 0.00 mm
- net FIRE: track 32.7 -> 0.00 mm
- net PADDLE_A: track 26.8 -> 0.00 mm
- net TRIGGER1: track 0.00 -> 26.5 mm
- net Net-(D1-Pad1): track 0.00 -> 24.7 mm
- net TRIGGER2: track 0.00 -> 21.1 mm
- net Net-(J2-Pad7): track 0.00 -> 19.7 mm
- net PADDLE_B: track 16.8 -> 0.00 mm
- net /MD_BTN_B: track 15.4 -> 0.00 mm
- net VCC: track 38.6 -> 24.7 mm, vias 1 -> 0
- net Net-(D2-Pad1): track 0.00 -> 12.2 mm
- net OUT: track 0.00 -> 10.9 mm
- net Net-(Q2-Pad2): track 6.50 -> 0.00 mm
- net Net-(Q1-Pad2): track 6.50 -> 0.00 mm
- net DOWN: track 20.3 -> 22.6 mm
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Other:
- net class Power added: clearance 0.2, trace_width 0.381, via_dia 0.6, via_drill 0.4
- board text added: "MSX"
- board text added: "MSX Mega Adapter"
- board text removed: "ATARI 7800"
- board text removed: "Atari 7800 MEGA Adapter"
- board text removed: "Revision A"

Commit message: Updated gerbers
Other:
- rule pad_to_mask_clearance: 0.2 -> 0
